Commit message: commit

File: husky_description/urdf/husky.urdf.xacro (robot description, xacro)
@@ -94,5 +94,5 @@
       <origin xyz="0 0 0" rpy="0.0 0.00 1.5708" />
       <geometry>
-        <box size="0.03 0.03 0.01" />
+        <box size="0.05 0.05 0.01" />
       </geometry >
       <material name="Apriltag36_11_00000">
@@ -116,5 +116,5 @@
 <!-- tag1 -->
   <joint name="tag1_joint" type="fixed">
-    <origin xyz = "0.15 0.05 0.26" rpy="0 0 0"/>
+    <origin xyz = "0.2 0.1 0.26" rpy="0 0 0"/>
     <parent link="base_link" />
     <child link="tag1" />
@@ -124,5 +124,5 @@
       <origin xyz="0 0 0" rpy="0.00 0.00 1.5708" />
       <geometry>
-        <box size="0.06 0.06 0.01" />
+        <box size="0.15 0.15 0.01" />
       </geometry >
       <material name="Apriltag36_11_00001">
@@ -145,5 +145,5 @@
 <!-- tag2 -->
   <joint name="tag2_joint" type="fixed">
-    <origin xyz = "0.15 -0.05 0.26" rpy="0 0 0"/>
+    <origin xyz = "0.2 -0.1 0.26" rpy="0 0 0"/>
     <parent link="base_link" />
     <child link="tag2" />
@@ -153,5 +153,5 @@
       <origin xyz="0 0 0" rpy="0.0 0.00 1.5708" />
       <geometry>
-        <box size="0.06 0.06 0.01" />
+        <box size="0.15 0.15 0.01" />
       </geometry >
       <material name="Apriltag36_11_00002">
@@ -174,5 +174,5 @@
 <!-- tag3 -->
   <joint name="tag3_joint" type="fixed">
-    <origin xyz = "0.05 -0.05 0.26" rpy="0 0 0"/>
+    <origin xyz = "0.0 -0.10 0.26" rpy="0 0 0"/>
     <parent link="base_link" />
     <child link="tag3" />
@@ -182,5 +182,5 @@
       <origin xyz="0 0 0" rpy="0.0 0.00 1.5708" />
       <geometry>
-        <box size="0.06 0.06 0.01" />
+        <box size="0.15 0.15 0.01" />
       </geometry >
       <material name="Apriltag36_11_00003">
@@ -203,5 +203,5 @@
 <!-- tag4 -->
   <joint name="tag4_joint" type="fixed">
-    <origin xyz = "0.05 0.05 0.26" rpy="0 0 0"/>
+    <origin xyz = "0.00 0.10 0.26" rpy="0 0 0"/>
     <parent link="base_link" />
     <child link="tag4" />
@@ -211,5 +211,5 @@
       <origin xyz="0 0 0" rpy="0.0 0.00 1.5708" />
       <geometry>
-        <box size="0.06 0.06 0.01" />
+        <box size="0.15 0.15 0.01" />
       </geometry >
       <material name="Apriltag36_11_00004">
@@ -229,236 +229,4 @@
   <gazebo reference="tag4">
     <material>Apriltag36_11_00004</material>
-  </gazebo>
-<!-- tag5 -->
-  <joint name="tag5_joint" type="fixed">
-    <origin xyz = "0.25 0.15 0.26" rpy="0 0 0"/>
-    <parent link="base_link" />
-    <child link="tag5" />
-  </joint>
-  <link name="tag5">
-    <visual>
-      <origin xyz="0 0 0" rpy="0.0 0.00 1.5708" />
-      <geometry>
-        <box size="0.10 0.10 0.01" />
-      </geometry >
-      <material name="Apriltag36_11_00005">
-        <script>
-          <uri>file://./Apriltag36_11_00005/materials/scripts</uri>
-          <uri>file://./Apriltag36_11_00005/materials/textures</uri>
-          <name>Apriltag36_11_00005</name>
-        </script>
-      </material>
-    </visual>
-    <inertial>
-      <origin xyz="0 0 0"/>
-      <mass value="0.1" />
-      <inertia ixx="0.01" ixy="0.0" ixz="0.0" iyy="0.01" iyz="0.0" izz="0.01"/>
-    </inertial>
-  </link>
-  <gazebo reference="tag5">
-    <material>Apriltag36_11_00005</material>
-  </gazebo>
-<!-- tag6 -->
-  <joint name="tag6_joint" type="fixed">
-    <origin xyz = "0.25 -0.15 0.26" rpy="0 0 0"/>
-    <parent link="base_link" />
-    <child link="tag6" />
-  </joint>
-  <link name="tag6">
-    <visual>
-      <origin xyz="0 0 0" rpy="0.0 0.00 1.5708" />
-      <geometry>
-        <box size="0.10 0.10 0.01" />
-      </geometry >
-      <material name="Apriltag36_11_00006">
-        <script>
-          <uri>file://./Apriltag36_11_00006/materials/scripts</uri>
-          <uri>file://./Apriltag36_11_00006/materials/textures</uri>
-          <name>Apriltag36_11_00006</name>
-        </script>
-      </material>
-    </visual>
-    <inertial>
-      <origin xyz="0 0 0"/>
-      <mass value="0.1" />
-      <inertia ixx="0.01" ixy="0.0" ixz="0.0" iyy="0.01" iyz="0.0" izz="0.01"/>
-    </inertial>
-  </link>
-  <gazebo reference="tag6">
-    <material>Apriltag36_11_00006</material>
-  </gazebo>
-<!-- tag7 -->
-  <joint name="tag7_joint" type="fixed">
-    <origin xyz = "-0.05 -0.15 0.26" rpy="0 0 0"/>
-    <parent link="base_link" />
-    <child link="tag7" />
-  </joint>
-  <link name="tag7">
-    <visual>
-      <origin xyz="0 0 0" rpy="0.0 0.00 1.5708" />
-      <geometry>
-        <box size="0.10 0.10 0.01" />
-      </geometry >
-      <material name="Apriltag36_11_00007">
-        <script>
-          <uri>file://./Apriltag36_11_00007/materials/scripts</uri>
-          <uri>file://./Apriltag36_11_00007/materials/textures</uri>
-          <name>Apriltag36_11_00007</name>
-        </script>
-      </material>
-    </visual>
-    <inertial>
-      <origin xyz="0 0 0"/>
-      <mass value="0.1" />
-      <inertia ixx="0.01" ixy="0.0" ixz="0.0" iyy="0.01" iyz="0.0" izz="0.01"/>
-    </inertial>
-  </link>
-  <gazebo reference="tag7">
-    <material>Apriltag36_11_00007</material>
-  </gazebo>
-<!-- tag8 -->
-  <joint name="tag8_joint" type="fixed">
-    <origin xyz = "-0.05 0.15 0.26" rpy="0 0 0"/>
-    <parent link="base_link" />
-    <child link="tag8" />
-  </joint>
-  <link name="tag8">
-    <visual>
-      <origin xyz="0 0 0" rpy="0.0 0.00 1.5708" />
-      <geometry>
-        <box size="0.10 0.1 0.01" />
-      </geometry >
-      <material name="Apriltag36_11_00008">
-        <script>
-          <uri>file://./Apriltag36_11_00008/materials/scripts</uri>
-          <uri>file://./Apriltag36_11_00008/materials/textures</uri>
-          <name>Apriltag36_11_00008</name>
-        </script>
-      </material>
-    </visual>
-    <inertial>
-      <origin xyz="0 0 0"/>
-      <mass value="0.1" />
-      <inertia ixx="0.01" ixy="0.0" ixz="0.0" iyy="0.01" iyz="0.0" izz="0.01"/>
-    </inertial>
-  </link>
-  <gazebo reference="tag8">
-    <material>Apriltag36_11_00008</material>
-  </gazebo>
-  <!-- tag9 -->
-  <joint name="tag9_joint" type="fixed">
-    <origin xyz = "0.25 0.0 0.26" rpy="0 0 0"/>
-    <parent link="base_link" />
-    <child link="tag9" />
-  </joint>
-  <link name="tag9">
-    <visual>
-      <origin xyz="0 0 0" rpy="0.0 0.00 1.5708" />
-      <geometry>
-        <box size="0.10 0.10 0.01" />
-      </geometry >
-      <material name="Apriltag36_11_00009">
-        <script>
-          <uri>file://./Apriltag36_11_00009/materials/scripts</uri>
-          <uri>file://./Apriltag36_11_00009/materials/textures</uri>
-          <name>Apriltag36_11_00009</name>
-        </script>
-      </material>
-    </visual>
-    <inertial>
-      <origin xyz="0 0 0"/>
-      <mass value="0.1" />
-      <inertia ixx="0.01" ixy="0.0" ixz="0.0" iyy="0.01" iyz="0.0" izz="0.01"/>
-    </inertial>
-  </link>
-  <gazebo reference="tag9">
-    <material>Apriltag36_11_00009</material>
-  </gazebo>
-<!-- tag10 -->
-  <joint name="tag10_joint" type="fixed">
-    <origin xyz = "0.1 -0.15 0.26" rpy="0 0 0"/>
-    <parent link="base_link" />
-    <child link="tag10" />
-  </joint>
-  <link name="tag10">
-    <visual>
-      <origin xyz="0 0 0" rpy="0.0 0.00 1.5708" />
-      <geometry>
-        <box size="0.10 0.1 0.01" />
-      </geometry >
-      <material name="Apriltag36_11_00010">
-        <script>
-          <uri>file://./Apriltag36_11_00010/materials/scripts</uri>
-          <uri>file://./Apriltag36_11_00010/materials/textures</uri>
-          <name>Apriltag36_11_00010</name>
-        </script>
-      </material>
-    </visual>
-    <inertial>
-      <origin xyz="0 0 0"/>
-      <mass value="0.1" />
-      <inertia ixx="0.01" ixy="0.0" ixz="0.0" iyy="0.01" iyz="0.0" izz="0.01"/>
-    </inertial>
-  </link>
-  <gazebo reference="tag10">
-    <material>Apriltag36_11_00010</material>
-  </gazebo>
-<!-- tag11 -->
-  <joint name="tag11_joint" type="fixed">
-    <origin xyz = "-0.05 0.0 0.26" rpy="0 0 0"/>
-    <parent link="base_link" />
-    <child link="tag11" />
-  </joint>
-  <link name="tag11">
-    <visual>
-      <origin xyz="0 0 0" rpy="0.0 0.00 1.5708" />
-      <geometry>
-        <box size="0.11 0.1 0.01" />
-      </geometry >
-      <material name="Apriltag36_11_00011">
-        <script>
-          <uri>file://./Apriltag36_11_00011/materials/scripts</uri>
-          <uri>file://./Apriltag36_11_00011/materials/textures</uri>
-          <name>Apriltag36_11_00011</name>
-        </script>
-      </material>
-    </visual>
-    <inertial>
-      <origin xyz="0 0 0"/>
-      <mass value="0.1" />
-      <inertia ixx="0.01" ixy="0.0" ixz="0.0" iyy="0.01" iyz="0.0" izz="0.01"/>
-    </inertial>
-  </link>
-  <gazebo reference="tag11">
-    <material>Apriltag36_11_00011</material>
-  </gazebo>
-<!-- tag12 -->
-  <joint name="tag12_joint" type="fixed">
-    <origin xyz = "0.1 0.150 0.26" rpy="0 0 0"/>
-    <parent link="base_link" />
-    <child link="tag12" />
-  </joint>
-  <link name="tag12">
-    <visual>
-      <origin xyz="0 0 0" rpy="0.0 0.00 1.5708" />
-      <geometry>
-        <box size="0.10 0.1 0.01" />
-      </geometry >
-      <material name="Apriltag36_11_00012">
-        <script>
-          <uri>file://./Apriltag36_11_00012/materials/scripts</uri>
-          <uri>file://./Apriltag36_11_00012/materials/textures</uri>
-          <name>Apriltag36_11_00012</name>
-        </script>
-      </material>
-    </visual>
-    <inertial>
-      <origin xyz="0 0 0"/>
-      <mass value="0.1" />
-      <inertia ixx="0.01" ixy="0.0" ixz="0.0" iyy="0.01" iyz="0.0" izz="0.01"/>
-    </inertial>
-  </link>
-  <gazebo reference="tag12">
-    <material>Apriltag36_11_00012</material>
   </gazebo>
   <!-- Base footprint is on the ground under the robot -->

Commit message: clean

File: husky_description/urdf/husky.urdf.xacro (robot description, xacro)
@@ -92,5 +92,5 @@
   <link name="tag0">
     <visual>
-      <origin xyz="0 0 0" rpy="0.0 0.00 1.5708" />
+      <origin xyz="0 0 0" rpy="0.00 0.00 1.5708" />
       <geometry>
         <box size="0.03 0.03 0.01" />
@@ -151,5 +151,5 @@
   <link name="tag2">
     <visual>
-      <origin xyz="0 0 0" rpy="0.0 0.00 1.5708" />
+      <origin xyz="0 0 0" rpy="0.00 0.00 1.5708" />
       <geometry>
         <box size="0.06 0.06 0.01" />
@@ -180,5 +180,5 @@
   <link name="tag3">
     <visual>
-      <origin xyz="0 0 0" rpy="0.0 0.00 1.5708" />
+      <origin xyz="0 0 0" rpy="0.00 0.00 1.5708" />
       <geometry>
         <box size="0.06 0.06 0.01" />
@@ -209,5 +209,5 @@
   <link name="tag4">
     <visual>
-      <origin xyz="0 0 0" rpy="0.0 0.00 1.5708" />
+      <origin xyz="0 0 0" rpy="0.00 0.00 1.5708" />
       <geometry>
         <box size="0.06 0.06 0.01" />
@@ -238,5 +238,5 @@
   <link name="tag5">
     <visual>
-      <origin xyz="0 0 0" rpy="0.0 0.00 1.5708" />
+      <origin xyz="0 0 0" rpy="0.00 0.00 1.5708" />
       <geometry>
         <box size="0.10 0.10 0.01" />
@@ -267,5 +267,5 @@
   <link name="tag6">
     <visual>
-      <origin xyz="0 0 0" rpy="0.0 0.00 1.5708" />
+      <origin xyz="0 0 0" rpy="0.00 0.00 1.5708" />
       <geometry>
         <box size="0.10 0.10 0.01" />
@@ -296,5 +296,5 @@
   <link name="tag7">
     <visual>
-      <origin xyz="0 0 0" rpy="0.0 0.00 1.5708" />
+      <origin xyz="0 0 0" rpy="0.00 0.00 1.5708" />
       <geometry>
         <box size="0.10 0.10 0.01" />
@@ -325,5 +325,5 @@
   <link name="tag8">
     <visual>
-      <origin xyz="0 0 0" rpy="0.0 0.00 1.5708" />
+      <origin xyz="0 0 0" rpy="0.00 0.00 1.5708" />
       <geometry>
         <box size="0.10 0.1 0.01" />
@@ -354,5 +354,5 @@
   <link name="tag9">
     <visual>
-      <origin xyz="0 0 0" rpy="0.0 0.00 1.5708" />
+      <origin xyz="0 0 0" rpy="0.00 0.00 1.5708" />
       <geometry>
         <box size="0.10 0.10 0.01" />
@@ -383,5 +383,5 @@
   <link name="tag10">
     <visual>
-      <origin xyz="0 0 0" rpy="0.0 0.00 1.5708" />
+      <origin xyz="0 0 0" rpy="0.00 0.00 1.5708" />
       <geometry>
         <box size="0.10 0.1 0.01" />
@@ -412,5 +412,5 @@
   <link name="tag11">
     <visual>
-      <origin xyz="0 0 0" rpy="0.0 0.00 1.5708" />
+      <origin xyz="0 0 0" rpy="0.00 0.00 1.5708" />
       <geometry>
         <box size="0.11 0.1 0.01" />
@@ -441,5 +441,5 @@
   <link name="tag12">
     <visual>
-      <origin xyz="0 0 0" rpy="0.0 0.00 1.5708" />
+      <origin xyz="0 0 0" rpy="0.00 0.00 1.5708" />
       <geometry>
         <box size="0.10 0.1 0.01" />

Commit message: tag position

File: husky_description/urdf/husky.urdf.xacro (robot description, xacro)
@@ -92,5 +92,5 @@
   <link name="tag0">
     <visual>
-      <origin xyz="0 0 0" rpy="0.00 0.00 1.5708" />
+      <origin xyz="0 0 -0.005" rpy="0.00 0.00 1.5708" />
       <geometry>
         <box size="0.03 0.03 0.01" />
@@ -122,5 +122,5 @@
   <link name="tag1">
     <visual>
-      <origin xyz="0 0 0" rpy="0.00 0.00 1.5708" />
+      <origin xyz="0 0 -0.005" rpy="0.00 0.00 1.5708" />
       <geometry>
         <box size="0.06 0.06 0.01" />
@@ -151,5 +151,5 @@
   <link name="tag2">
     <visual>
-      <origin xyz="0 0 0" rpy="0.00 0.00 1.5708" />
+      <origin xyz="0 0 -0.005" rpy="0.00 0.00 1.5708" />
       <geometry>
         <box size="0.06 0.06 0.01" />
@@ -180,5 +180,5 @@
   <link name="tag3">
     <visual>
-      <origin xyz="0 0 0" rpy="0.00 0.00 1.5708" />
+      <origin xyz="0 0 -0.005" rpy="0.00 0.00 1.5708" />
       <geometry>
         <box size="0.06 0.06 0.01" />
@@ -209,5 +209,5 @@
   <link name="tag4">
     <visual>
-      <origin xyz="0 0 0" rpy="0.00 0.00 1.5708" />
+      <origin xyz="0 0 -0.005" rpy="0.00 0.00 1.5708" />
       <geometry>
         <box size="0.06 0.06 0.01" />
@@ -238,5 +238,5 @@
   <link name="tag5">
     <visual>
-      <origin xyz="0 0 0" rpy="0.00 0.00 1.5708" />
+      <origin xyz="0 0 -0.005" rpy="0.00 0.00 1.5708" />
       <geometry>
         <box size="0.10 0.10 0.01" />
@@ -267,5 +267,5 @@
   <link name="tag6">
     <visual>
-      <origin xyz="0 0 0" rpy="0.00 0.00 1.5708" />
+      <origin xyz="0 0 -0.005" rpy="0.00 0.00 1.5708" />
       <geometry>
         <box size="0.10 0.10 0.01" />
@@ -296,5 +296,5 @@
   <link name="tag7">
     <visual>
-      <origin xyz="0 0 0" rpy="0.00 0.00 1.5708" />
+      <origin xyz="0 0 -0.005" rpy="0.00 0.00 1.5708" />
       <geometry>
         <box size="0.10 0.10 0.01" />
@@ -325,5 +325,5 @@
   <link name="tag8">
     <visual>
-      <origin xyz="0 0 0" rpy="0.00 0.00 1.5708" />
+      <origin xyz="0 0 -0.005" rpy="0.00 0.00 1.5708" />
       <geometry>
         <box size="0.10 0.1 0.01" />
@@ -354,5 +354,5 @@
   <link name="tag9">
     <visual>
-      <origin xyz="0 0 0" rpy="0.00 0.00 1.5708" />
+      <origin xyz="0 0 -0.005" rpy="0.00 0.00 1.5708" />
       <geometry>
         <box size="0.10 0.10 0.01" />
@@ -383,5 +383,5 @@
   <link name="tag10">
     <visual>
-      <origin xyz="0 0 0" rpy="0.00 0.00 1.5708" />
+      <origin xyz="0 0 -0.005" rpy="0.00 0.00 1.5708" />
       <geometry>
         <box size="0.10 0.1 0.01" />
@@ -412,5 +412,5 @@
   <link name="tag11">
     <visual>
-      <origin xyz="0 0 0" rpy="0.00 0.00 1.5708" />
+      <origin xyz="0 0 -0.005" rpy="0.00 0.00 1.5708" />
       <geometry>
         <box size="0.11 0.1 0.01" />
@@ -441,5 +441,5 @@
   <link name="tag12">
     <visual>
-      <origin xyz="0 0 0" rpy="0.00 0.00 1.5708" />
+      <origin xyz="0 0 -0.005" rpy="0.00 0.00 1.5708" />
       <geometry>
         <box size="0.10 0.1 0.01" />
